Commit message: moveit able to plan and execute sometimes

File: Allegro_moveit_config/config/allegro_hand_right.ros2_control.xacro (robot description, xacro)
@@ -1,3 +1,3 @@
-<?xml version="1.0"?>
+<?xml version="1"?>
 <robot xmlns:xacro="http://www.ros.org/wiki/xacro">
     <xacro:macro name="allegro_hand_right_ros2_control" params="name initial_positions_file">
@@ -8,129 +8,129 @@
                 <plugin>mock_components/GenericSystem</plugin>
             </hardware>
-            <joint name="joint_0.0">
+            <joint name="joint_0">
                 <command_interface name="position"/>
                 <command_interface name="velocity"/>
                 <state_interface name="position">
-                  <param name="initial_value">${initial_positions['joint_0.0']}</param>
+                  <param name="initial_value">${initial_positions['joint_0']}</param>
                 </state_interface>
                 <state_interface name="velocity"/>
             </joint>
-            <joint name="joint_1.0">
+            <joint name="joint_1">
                 <command_interface name="position"/>
                 <command_interface name="velocity"/>
                 <state_interface name="position">
-                  <param name="initial_value">${initial_positions['joint_1.0']}</param>
+                  <param name="initial_value">${initial_positions['joint_1']}</param>
                 </state_interface>
                 <state_interface name="velocity"/>
             </joint>
-            <joint name="joint_2.0">
+            <joint name="joint_2">
                 <command_interface name="position"/>
                 <command_interface name="velocity"/>
                 <state_interface name="position">
-                  <param name="initial_value">${initial_positions['joint_2.0']}</param>
+                  <param name="initial_value">${initial_positions['joint_2']}</param>
                 </state_interface>
                 <state_interface name="velocity"/>
             </joint>
-            <joint name="joint_3.0">
+            <joint name="joint_3">
                 <command_interface name="position"/>
                 <command_interface name="velocity"/>
                 <state_interface name="position">
-                  <param name="initial_value">${initial_positions['joint_3.0']}</param>
+                  <param name="initial_value">${initial_positions['joint_3']}</param>
                 </state_interface>
                 <state_interface name="velocity"/>
             </joint>
-            <joint name="joint_12.0">
+            <joint name="joint_12">
                 <command_interface name="position"/>
                 <command_interface name="velocity"/>
                 <state_interface name="position">
-                  <param name="initial_value">${initial_positions['joint_12.0']}</param>
+                  <param name="initial_value">${initial_positions['joint_12']}</param>
                 </state_interface>
                 <state_interface name="velocity"/>
             </joint>
-            <joint name="joint_13.0">
+            <joint name="joint_13">
                 <command_interface name="position"/>
                 <command_interface name="velocity"/>
                 <state_interface name="position">
-                  <param name="initial_value">${initial_positions['joint_13.0']}</param>
+                  <param name="initial_value">${initial_positions['joint_13']}</param>
                 </state_interface>
                 <state_interface name="velocity"/>
             </joint>
-            <joint name="joint_14.0">
+            <joint name="joint_14">
                 <command_interface name="position"/>
                 <command_interface name="velocity"/>
                 <state_interface name="position">
-                  <param name="initial_value">${initial_positions['joint_14.0']}</param>
+                  <param name="initial_value">${initial_positions['joint_14']}</param>
                 </state_interface>
                 <state_interface name="velocity"/>
             </joint>
-            <joint name="joint_15.0">
+            <joint name="joint_15">
                 <command_interface name="position"/>
                 <command_interface name="velocity"/>
                 <state_interface name="position">
-                  <param name="initial_value">${initial_positions['joint_15.0']}</param>
+                  <param name="initial_value">${initial_positions['joint_15']}</param>
                 </state_interface>
                 <state_interface name="velocity"/>
             </joint>
-            <joint name="joint_4.0">
+            <joint name="joint_4">
                 <command_interface name="position"/>
                 <command_interface name="velocity"/>
                 <state_interface name="position">
-                  <param name="initial_value">${initial_positions['joint_4.0']}</param>
+                  <param name="initial_value">${initial_positions['joint_4']}</param>
                 </state_interface>
                 <state_interface name="velocity"/>
             </joint>
-            <joint name="joint_5.0">
+            <joint name="joint_5">
                 <command_interface name="position"/>
                 <command_interface name="velocity"/>
                 <state_interface name="position">
-                  <param name="initial_value">${initial_positions['joint_5.0']}</param>
+                  <param name="initial_value">${initial_positions['joint_5']}</param>
                 </state_interface>
                 <state_interface name="velocity"/>
             </joint>
-            <joint name="joint_6.0">
+            <joint name="joint_6">
                 <command_interface name="position"/>
                 <command_interface name="velocity"/>
                 <state_interface name="position">
-                  <param name="initial_value">${initial_positions['joint_6.0']}</param>
+                  <param name="initial_value">${initial_positions['joint_6']}</param>
                 </state_interface>
                 <state_interface name="velocity"/>
             </joint>
-            <joint name="joint_7.0">
+            <joint name="joint_7">
                 <command_interface name="position"/>
                 <command_interface name="velocity"/>
                 <state_interface name="position">
-                  <param name="initial_value">${initial_positions['joint_7.0']}</param>
+                  <param name="initial_value">${initial_positions['joint_7']}</param>
                 </state_interface>
                 <state_interface name="velocity"/>
             </joint>
-            <joint name="joint_8.0">
+            <joint name="joint_8">
                 <command_interface name="position"/>
                 <command_interface name="velocity"/>
                 <state_interface name="position">
-                  <param name="initial_value">${initial_positions['joint_8.0']}</param>
+                  <param name="initial_value">${initial_positions['joint_8']}</param>
                 </state_interface>
                 <state_interface name="velocity"/>
             </joint>
-            <joint name="joint_9.0">
+            <joint name="joint_9">
                 <command_interface name="position"/>
                 <command_interface name="velocity"/>
                 <state_interface name="position">
-                  <param name="initial_value">${initial_positions['joint_9.0']}</param>
+                  <param name="initial_value">${initial_positions['joint_9']}</param>
                 </state_interface>
                 <state_interface name="velocity"/>
             </joint>
-            <joint name="joint_10.0">
+            <joint name="joint_10">
                 <command_interface name="position"/>
                 <command_interface name="velocity"/>
                 <state_interface name="position">
-                  <param name="initial_value">${initial_positions['joint_10.0']}</param>
+                  <param name="initial_value">${initial_positions['joint_10']}</param>
                 </state_interface>
                 <state_interface name="velocity"/>
             </joint>
-            <joint name="joint_11.0">
+            <joint name="joint_11">
                 <command_interface name="position"/>
                 <command_interface name="velocity"/>
                 <state_interface name="position">
-                  <param name="initial_value">${initial_positions['joint_11.0']}</param>
+                  <param name="initial_value">${initial_positions['joint_11']}</param>
                 </state_interface>
                 <state_interface name="velocity"/>

File: control_hand/urdf/AllegroHandRight.urdf.xacro (robot description, xacro)
@@ -100,5 +100,5 @@
             </inertial>
         </link>
-        <joint name="joint_${finger_num*4+0}.0" type="revolute">
+        <joint name="joint_${finger_num*4+0}" type="revolute">
             <axis xyz="-1 0 0"/>
             <limit effort="15" velocity="7"
@@ -135,5 +135,5 @@
             </inertial>
         </link>
-        <joint name="joint_${finger_num*4+1}.0" type="revolute">
+        <joint name="joint_${finger_num*4+1}" type="revolute">
             <axis xyz="0 0 1"/>
             <limit effort="15" velocity="7"
@@ -167,5 +167,5 @@
             </inertial>
         </link>
-        <joint name="joint_${finger_num*4+2}.0" type="revolute">
+        <joint name="joint_${finger_num*4+2}" type="revolute">
             <axis xyz="0 1 0"/>
             <limit effort="15" velocity="7"
@@ -200,5 +200,5 @@
             </inertial>
         </link>
-        <joint name="joint_${finger_num*4+3}.0" type="revolute">
+        <joint name="joint_${finger_num*4+3}" type="revolute">
             <axis xyz="0 1 0"/>
             <limit effort="15" velocity="7"
@@ -266,5 +266,5 @@
             </inertial>
         </link>
-        <joint name="joint_${finger_num*4+0}.0" type="revolute">
+        <joint name="joint_${finger_num*4+0}" type="revolute">
             <axis xyz="0 0 1"/>
             <limit effort="15" velocity="7"
@@ -299,5 +299,5 @@
             </inertial>
         </link>
-        <joint name="joint_${finger_num*4+1}.0" type="revolute">
+        <joint name="joint_${finger_num*4+1}" type="revolute">
             <limit effort="15" velocity="7"
                    lower="${limit_1_low+joint_safety_margin}"
@@ -331,5 +331,5 @@
             </inertial>
         </link>
-        <joint name="joint_${finger_num*4+2}.0" type="revolute">
+        <joint name="joint_${finger_num*4+2}" type="revolute">
             <axis xyz="0 1 0"/>
             <limit effort="15" velocity="7"
@@ -363,5 +363,5 @@
             </inertial>
         </link>
-        <joint name="joint_${finger_num*4+3}.0" type="revolute">
+        <joint name="joint_${finger_num*4+3}" type="revolute">
             <axis xyz="0 1 0"/>
             <limit effort="15" velocity="7"
